File: electronics/kicad/mk-brace-sensing.kicad_sch (KiCad schematic)
At the start: 28 parts, among them J1 Harness, hinge end, J2 Calf FSRs, J3 Harness, thigh end, SW1 Power, U1 XIAO ESP32-S3, U2 AS5600, U3 LSM6DSOX, U4 LSM6DSOX

Commit message: Schematic rev B (WIP): power path, AS5600 DIR, FSR ADC range
From an external design review, checked against the AS5600 and ESP32-S3
datasheets:
- SW1 and a 0.5 A PTC (F1) moved to the cell on the thigh side, so the
  harness carries no battery voltage when off and is short-protected
- AS5600 DIR tied to GND (must not float); D7 freed
- 1.5k series resistors on each FSR line keep the ADC input <= 2.87 V
  (ESP32-S3 12 dB range is 0-2.9 V) and limit harness fault current
ERC 0 errors; netlist re-checked. Remaining rev B items in HANDOFF.md.

Co-Authored-By: claude-flow <ruv@ruv.net>
Parts:
- added F1: PTC 0.5A hold, Fuse:Fuse_1206_3216Metric, symbol Device:Polyfuse
- added R10, R11, R12, R9: 1.5k, Resistor_SMD:R_0603_1608Metric, symbol Device:R
Connections:
- net FSR_C1: now also R11.1; no longer R3.1, U1.4 (D3/A3)
- net FSR_C2: now also R12.1; no longer R4.1, U1.9 (D8/A8)
- net FSR_T1: now also R9.1; no longer R1.1, U1.1 (D0/A0)
- net FSR_T2: now also R10.1; no longer R2.1, U1.2 (D1/A1)
- net GND: now also U2.8 (DIR)
- net VBAT_SW: now also J1.1 (Pin_1), J3.1 (Pin_1)
- net ENC_DIR: no longer names the net of U1.8 (D7/RX)
- net ENC_DIR: no longer U2.8 (DIR)
- removed net VBAT_RAW: BT1.1 (+), J1.1 (Pin_1), J3.1 (Pin_1), SW1.1 (A)
- new net FSR_C1_ADC: R11.2, R3.1, U1.4 (D3/A3)
- new net FSR_C2_ADC: R12.2, R4.1, U1.9 (D8/A8)
- new net FSR_T1_ADC: R1.1, R9.2, U1.1 (D0/A0)
- new net FSR_T2_ADC: R10.2, R2.1, U1.2 (D1/A1)
- new net VBAT_CELL: BT1.1 (+), F1.1
- new net VBAT_FUSED: F1.2, SW1.1 (A)
- no-connect marks 11 -> 12
Other:
- note added: "Battery protection: cell PCM + F1 PTC + SW1, all at the cell"
- note added: "FSR series resistors (keep ADC input <= 2.87 V, limit harness fault current)"
- note added: "Notes: 1. I2C bus: AS5600 0x36, shin IMU 0x6B (SA0 high), thigh IMU 0x6A (SA0 low). 2.2k pull-ups on the hinge board only. 2. FSRs: FSR_EN drives the top of all four dividers, high only while sampling. Out = 3.3 V x 10k / (10k + 1.5k + R_fsr) <= 2.87 V, inside the 0-2.9 V ADC range at 12 dB. All on ADC1. Relative contact indication only, not calibrated pressure. 3. VBAT_SENSE = VBAT_SW / 2 (220k/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"
- note removed: "Notes: 1. I2C bus: AS5600 0x36, shin IMU 0x6B (SA0 high), thigh IMU 0x6A (SA0 low). 2.2k pull-ups on the hinge board only. 2. FSRs: FSR_EN drives the top of all four dividers, high only while sampling. Out = 10k / (10k + R_fsr) x 3.3 V. All on ADC1. 3. VBAT_SENSE = VBAT_SW / 2 (220k/220k, ~10 uA). Firmware cutoff 3.5 V. 4. Thigh IMU INT is not routed (harness kept to 8 conductors); poll it over I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"
- moved on the sheet: SW1
